File: pcb/KiBot-CICD-Template.kicad_sch (KiCad schematic)
At the start: 1 part

Commit message: Set initial project defaults
Signed-off-by: Terry Cox <terry@bootstrap.je>
Other:
- company: nerdyscout -> Bootstrap Ltd
Changed lines of the file:
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@@
     (date "${date}")
     (rev "${version}")
-    (company "nerdyscout")
+    (company "Bootstrap Ltd")
     (comment 4 "CERN Open Hardware Licence v2.0")
   )
