File: pcb/KiBot-CICD-Template.kicad_pcb (KiCad board)
At the start: 4 copper layers, 30.5 x 17.8 mm, 0 parts

Commit message: Set initial project defaults
Signed-off-by: Terry Cox <terry@bootstrap.je>
Routing:
- removed copper zone on In1.Cu, net (none)
- removed copper zone on In2.Cu, net (none)
Other:
- copper layers 4 -> 2
Changed lines of the file:
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@@
 (kicad_pcb (version 20211014) (generator pcbnew)
   (general
-    (thickness 0.8)
+    (thickness 1.6)
   )
   (paper "A4")
@@
     (date "${date}")
     (rev "${version}")
-    (company "nerdyscout")
+    (company "Bootstrap Ltd")
     (comment 4 "CERN Open Hardware Licence v2.0")
   )
   (layers
     (0 "F.Cu" mixed)
-    (1 "In1.Cu" signal)
-    (2 "In2.Cu" signal)
     (31 "B.Cu" mixed)
     (32 "B.Adhes" user "B.Adhesive")
@@
     (48 "B.Fab" user)
     (49 "F.Fab" user)
+    (50 "User.1" user)
+    (51 "User.2" user)
+    (52 "User.3" user)
+    (53 "User.4" user)
+    (54 "User.5" user)
+    (55 "User.6" user)
+    (56 "User.7" user)
+    (57 "User.8" user)
+    (58 "User.9" user)
   )
   (setup
+    (stackup
+      (layer "F.SilkS" (type "Top Silk Screen") (color "White"))
+      (layer "F.Paste" (type "Top Solder Paste"))
+      (layer "F.Mask" (type "Top Solder Mask") (color "Green") (thickness 0.01))
+      (layer "F.Cu" (type "copper") (thickness 0.035))
+      (layer "dielectric 1" (type "core") (thickness 1.51) (material "FR4") (epsilon_r 4.5) (loss_tangent 0.02))
+      (layer "B.Cu" (type "copper") (thickness 0.035))
+      (layer "B.Mask" (type "Bottom Solder Mask") (color "Green") (thickness 0.01))
+      (layer "B.Paste" (type "Bottom Solder Paste"))
+      (layer "B.SilkS" (type "Bottom Silk Screen") (color "White"))
+      (copper_finish "None")
+      (dielectric_constraints no)
+    )
     (pad_to_mask_clearance 0)
     (aux_axis_origin 137.16 104.14)

Commit message: Refine DRC rules for 2-layer 1oz JLCPCB
Signed-off-by: Terry Cox <terry@bootstrap.je>
Other:
- rule pad_to_mask_clearance: 0 -> 0.05
Changed lines of the file:
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@@
       (layer "B.Paste" (type "Bottom Solder Paste"))
       (layer "B.SilkS" (type "Bottom Silk Screen") (color "White"))
-      (copper_finish "None")
+      (copper_finish "ENIG")
       (dielectric_constraints no)
     )
-    (pad_to_mask_clearance 0)
+    (pad_to_mask_clearance 0.05)
+    (solder_mask_min_width 0.254)
     (aux_axis_origin 137.16 104.14)
     (grid_origin 137.16 104.14)

Commit message: Migrated to KiCAD 8
Routing:
- removed copper zone on B.Cu, net (none)
- removed copper zone on F.Cu, net (none)
Other:
- board outline removed
- rule pad_to_mask_clearance: 0.05 -> 0
- board text removed: "${version}"
- board text removed: "KiBot-CICD-Template"
